File: Board_LDR/Board_LDR.kicad_sch (KiCad schematic)
At the start: 4 parts, among them J1 Conn_01x03, J2 Conn_01x04

Commit message: Elektromagnet kicad
Connections:
- net at J2.1 (Pin_1), R1.2: now also J1.2 (Pin_2)
- net at J2.2 (Pin_2): now also J1.3 (Pin_3), J2.4 (Pin_4); no longer J1.2 (Pin_2)
Changed lines of the file:
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@@
 	(paper "A4")
+	(junction
+		(at 121.92 72.39)
+		(diameter 0)
+		(color 0 0 0 0)
+	)
+	(junction
+		(at 118.11 81.28)
+		(diameter 0)
+		(color 0 0 0 0)
+	)
 	(junction
 		(at 113.03 67.31)
 		(diameter 0)
 		(color 0 0 0 0)
+	)
+	(wire
+		(pts
+			(xy 121.92 72.39) (xy 121.92 83.82)
+		)
+		(stroke
+			(width 0)
+			(type default)
+		)
 	)
 	(wire
@@
 	(wire
 		(pts
+			(xy 118.11 69.85) (xy 118.11 81.28)
+		)
+		(stroke
+			(width 0)
+			(type default)
+		)
+	)
+	(wire
+		(pts
 			(xy 119.38 88.9) (xy 119.38 72.39)
+		)
+		(stroke
+			(width 0)
+			(type default)
+		)
+	)
+	(wire
+		(pts
+			(xy 121.92 72.39) (xy 123.19 72.39)
 		)
 		(stroke
@@
 	(wire
 		(pts
-			(xy 119.38 72.39) (xy 123.19 72.39)
+			(xy 119.38 72.39) (xy 121.92 72.39)
 		)
 		(stroke
@@
 	(wire
 		(pts
-			(xy 113.03 81.28) (xy 123.19 81.28)
+			(xy 113.03 81.28) (xy 118.11 81.28)
 		)
 		(stroke
@@
 	(wire
 		(pts
-			(xy 121.92 69.85) (xy 123.19 69.85)
+			(xy 118.11 69.85) (xy 123.19 69.85)
 		)
 		(stroke
@@
 	(wire
 		(pts
-			(xy 121.92 83.82) (xy 121.92 69.85)
+			(xy 118.11 81.28) (xy 123.19 81.28)
 		)
 		(stroke
