File: KiCad_Elektromagnet/KiCad_Elektromagnet.kicad_sch (KiCad schematic)
At the start: 5 parts, among them J2 Conn_02x20_Counter_Clockwise_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, Q1 2N7000

Commit message: Elektromagnet kicad
Connections:
- net +5V renamed +12V
Other:
- note added: "0,5217391A"
- note added: "34,5 Ohm"
Changed lines of the file:
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@@
+		)
+	)
+	(text "0,5217391A"
+		(exclude_from_sim no)
+		(at 132.588 53.34 0)
+		(effects
+			(font
+				(size 1.27 1.27)
+			)
 		)
 	)
@@
 		(exclude_from_sim no)
 		(at 100.584 80.01 0)
+		(effects
+			(font
+				(size 1.27 1.27)
+			)
+		)
+	)
+	(text "34,5 Ohm\n"
+		(exclude_from_sim no)
+		(at 149.606 53.086 0)
 		(effects
 			(font
@@
 			)
 		)
-		(property "Value" "+5V"
+		(property "Value" "+12V"
 			(at 139.7 33.02 0)
 			(effects
