File: kiCad_LDR_flip_flop/kiCad_LDR_flip_flop.kicad_sch (KiCad schematic)
At the start: 10 parts, among them J1 Conn_01x02_MountingPin, J2 Conn_01x01_MountingPin, J3 Screw_Terminal_01x02, Q2 IRLZ34N

Commit message: made flip flop work
Parts:
- J2: footprint (none) -> Connector_PinSocket_2.54mm:PinSocket_1x01_P2.54mm_Vertical
Changed lines of the file:
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@@
 			)
 		)
-		(property "Footprint" ""
+		(property "Footprint" "Connector_PinSocket_2.54mm:PinSocket_1x01_P2.54mm_Vertical"
 			(at 130.81 86.36 0)
 			(effects

Commit message: KiCad changes
Parts:
- C1: value C -> 1 μF
- D1: value D -> 1N4002
- Op-amp2: renamed from Op-amp1; value MCP6001R -> MCP6002
- R1: value 65 ohm -> 24 ohm
Changed lines of the file:
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@@
 	(wire
 		(pts
-			(xy 186.69 124.46) (xy 186.69 140.97)
-		)
-		(stroke
-			(width 0)
-			(type default)
-		)
-	)
-	(wire
-		(pts
-			(xy 194.31 124.46) (xy 186.69 124.46)
+			(xy 189.23 124.46) (xy 189.23 132.08)
+		)
+		(stroke
+			(width 0)
+			(type default)
+		)
+	)
+	(wire
+		(pts
+			(xy 194.31 124.46) (xy 189.23 124.46)
 		)
 		(stroke
@@
 	(wire
 		(pts
-			(xy 180.34 140.97) (xy 180.34 132.08)
-		)
-		(stroke
-			(width 0)
-			(type default)
-		)
-	)
-	(wire
-		(pts
 			(xy 184.15 88.9) (xy 184.15 105.41)
 		)
@@
 	(wire
 		(pts
-			(xy 180.34 132.08) (xy 167.64 132.08)
-		)
-		(stroke
-			(width 0)
-			(type default)
-		)
-	)
-	(wire
-		(pts
-			(xy 186.69 140.97) (xy 180.34 140.97)
+			(xy 167.64 132.08) (xy 189.23 132.08)
 		)
 		(stroke
@@
 		(on_board yes)
 		(dnp no)
-		(fields_autoplaced yes)
 		(property "Reference" "#PWR08"
 			(at 115.57 110.49 0)
@@
 		)
 		(property "Value" "+3V3"
-			(at 115.57 119.38 0)
+			(at 114.046 118.872 0)
 			(effects
 				(font
@@
 		)
 		(property "Value" "+3V3"
-			(at 160.274 107.188 0)
+			(at 161.036 107.696 0)
 			(effects
 				(font
@@
 		(on_board yes)
 		(dnp no)
-		(fields_autoplaced yes)
 		(property "Reference" "#PWR09"
 			(at 118.11 120.65 0)
@@
 		)
 		(property "Value" "GND"
-			(at 118.11 119.38 0)
+			(at 120.396 118.618 0)
 			(effects
 				(font
@@
 		(on_board yes)
 		(dnp no)
-		(fields_autoplaced yes)
 		(property "Reference" "J1"
 			(at 201.93 122.2755 0)
@@
 		)
 		(property "Value" "Conn_01x02_MountingPin"
-			(at 201.93 124.8155 0)
+			(at 187.96 132.334 0)
 			(effects
 				(font
@@
 			)
 		)
-		(property "Value" "D"
+		(property "Value" "1N4002"
 			(at 179.07 85.09 0)
 			(effects
@@
 			)
 		)
-		(property "Value" "65 ohm"
+		(property "Value" "24 ohm"
 			(at 170.18 137.1599 0)
 			(effects
@@
 		(on_board yes)
 		(dnp no)
-		(property "Reference" "Op-amp1"
-			(at 163.068 83.058 0)
-			(effects
-				(font
-					(size 1.27 1.27)
-				)
-			)
-		)
-		(property "Value" "MCP6001R"
-			(at 160.274 89.154 0)
+		(property "Reference" "Op-amp2"
+			(at 146.304 103.632 0)
+			(effects
+				(font
+					(size 1.27 1.27)
+				)
+			)
+		)
+		(property "Value" "MCP6002"
+			(at 146.304 101.6 0)
 			(effects
 				(font
@@
 			(project "kiCad_LDR_flip_flop"
 				(path "/086cf29c-57f6-4286-ba50-433c4ba2e812"
-					(reference "Op-amp1")
+					(reference "Op-amp2")
 					(unit 1)
 				)
@@
 			)
 		)
-		(property "Value" "C"
+		(property "Value" "1 μF"
 			(at 189.23 83.82 90)
 			(effects
@@
 		)
 		(property "Value" "IRLZ34N"
-			(at 215.9 126.9999 0)
-			(effects
-				(font
+			(at 212.598 117.856 0)
+			(effects
+				(font
