File: kiCad_OLED_and_button/kiCad_OLED_and_button.kicad_pcb (KiCad board)
At the start: 2 copper layers, 6 parts, among them J1 OLED, J2 POWER and GND, J3 PICO pins, SW1 SW_Push, SW2 SW_Push, SW3 SW_Push

Commit message: kicad stuuf idk
Parts:
- moved J3 7.71 mm to (165.0, 107.5), turned to 180 degrees
Connections:
- J3 pad 1: Net-(J3-Pin_1) -> Net-(J1-SCK)
- J3 pad 2: Net-(J3-Pin_2) -> Net-(J1-SDA)
- J3 pad 4: Net-(J1-SDA) -> Net-(J3-Pin_4)
- J3 pad 5: Net-(J1-SCK) -> Net-(J3-Pin_5)
- SW1 pad 2: Net-(J3-Pin_1) -> Net-(J3-Pin_5)
- SW2 pad 2: Net-(J3-Pin_2) -> Net-(J3-Pin_4)
Routing:
- net Net-(J1-SCK): track 0.00 -> 52.5 mm
- net Net-(J1-SDA): track 0.00 -> 36.0 mm
- net Net-(J3-Pin_5): track 0.00 -> 28.6 mm
- net Net-(J3-Pin_3): track 6.50 -> 28.7 mm
- net GND: track 51.1 -> 69.1 mm
- net Net-(J3-Pin_4): track 0.00 -> 15.3 mm
- net Net-(J3-Pin_2): track 6.50 -> 0.00 mm
- net Net-(J3-Pin_1): track 6.50 -> 0.00 mm
Other:
- board outline added: 52.5 x 32.5 mm
