File: kiCad_LDRcomperator/LDRcomperator.kicad_sch (KiCad schematic)
At the start: 26 parts, among them J1 Screw_Terminal_01x02, J2 Conn_01x02_MountingPin, J3 Conn_01x02_MountingPin, J4 Conn_01x02_MountingPin, Q1 IRLZ34N

Commit message: Rapporten
Other:
- note added: "0.6 V (hvid)"
- note added: "1.5 V (sort)"
- note added: "1.8 V (sort)"
- note added: "2.7 V (hvid)"
Changed lines of the file:
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@@
+		)
+	)
+	(text "2.7 V (hvid)"
+		(exclude_from_sim no)
+		(at 91.694 118.872 0)
+		(effects
+			(font
+				(size 1.27 1.27)
+			)
+		)
+	)
+	(text "0.6 V (hvid)"
+		(exclude_from_sim no)
+		(at 89.662 90.932 0)
+		(effects
+			(font
+				(size 1.27 1.27)
+			)
+		)
+	)
+	(text "2.7 V (hvid)"
+		(exclude_from_sim no)
+		(at 100.076 105.664 0)
+		(effects
+			(font
+				(size 1.27 1.27)
+			)
+		)
+	)
+	(text "1.8 V (sort)"
+		(exclude_from_sim no)
+		(at 89.154 88.646 0)
+		(effects
+			(font
+				(size 1.27 1.27)
+			)
+		)
+	)
+	(text "1.5 V (sort)"
+		(exclude_from_sim no)
+		(at 99.822 107.95 0)
+		(effects
+			(font
+				(size 1.27 1.27)
+			)
 		)
 	)
@@
 		)
 	)
+	(text "1.5 V (sort)"
+		(exclude_from_sim no)
+		(at 91.44 116.078 0)
+		(effects
+			(font
+				(size 1.27 1.27)
+			)
+		)
+	)
 	(symbol
 		(lib_id "power:GND")
@@
 		(on_board yes)
 		(dnp no)
-		(fields_autoplaced yes)
 		(property "Reference" "#PWR08"
 			(at 97.79 90.17 0)
@@
 		)
 		(property "Value" "+3V3"
-			(at 97.79 99.06 0)
+			(at 97.79 98.044 0)
 			(effects
 				(font
@@
 		(on_board yes)
 		(dnp no)
-		(fields_autoplaced yes)
 		(property "Reference" "#PWR09"
 			(at 100.33 100.33 0)
@@
 		)
 		(property "Value" "GND"
-			(at 100.33 99.06 0)
-			(effects
-				(font
+			(at 102.616 98.044 0)
+			(effects
+				(font
