File: kiCad_LDRcomperator/_autosave-LDRcomperator.kicad_sch (KiCad schematic)
At the start: 26 parts, among them J1 Screw_Terminal_01x02, J2 Conn_01x02_MountingPin, J3 Conn_01x02_MountingPin, J4 Conn_01x02_MountingPin, Q1 BF244A

Commit message: Bare haft kigget på KiCad tegningerne
Parts:
- R2: value LDR03 -> LDR1
Changed lines of the file:
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@@
 		(on_board yes)
 		(dnp no)
-		(fields_autoplaced yes)
 		(property "Reference" "R3"
 			(at 139.7 83.8199 0)
@@
 		)
 		(property "Value" "2,2k ohm"
-			(at 139.7 86.3599 0)
+			(at 151.13 92.71 0)
 			(effects
 				(font
@@
 		(on_board yes)
 		(dnp no)
-		(fields_autoplaced yes)
 		(property "Reference" "#PWR03"
 			(at 137.16 64.77 0)
@@
 		)
 		(property "Value" "+3V3"
-			(at 137.16 55.88 0)
+			(at 137.16 57.15 0)
 			(effects
 				(font
@@
 			)
 		)
-		(property "Value" "LDR03"
+		(property "Value" "LDR1"
 			(at 139.7 69.8499 0)
 			(effects
